Commit message: Run the real-arm pipeline (lab_pick.py) end to end in Gazebo: --sim gazebo + scored rehearsal
- lab_pick --sim gazebo: Gazebo's MoveIt group and gripper_tcp, its trajectory
  controller, a 4x time allowance (Gazebo runs ~0.5x real time), and
  gazebo_rg2.py as the gripper (gripper action + grasp latch, latched only when
  the fingertips are at the block)
- planning group, controller and the 'gripper frame' test made configurable
  (any frame other than tool0 plans the gripper straight down)
- gazebo_pick_rehearsal.sh: starts everything with the windows open, resets the
  block (latch released first), runs the six scenarios, scores them against
  Gazebo's own block pose (gazebo_block_watch.py); software OpenGL by default
- world: saturated blue place pad; blue-grey soft gripper so the colour
  detector does not mistake it; 'absent or ambiguous' counts as not_found

Gazebo, keyword parser, GUI: 6/6 PASS (pick lifted to 0.187 m and set back;
place landed at (0.450, 0.201) on the pad).

Co-Authored-By: Claude Opus 5.5 <noreply@anthropic.com>

File: src/ur7e_bringup/urdf/dual_quick_changer.xacro (robot description, xacro)
@@ -57,5 +57,5 @@
         <origin xyz="0 0 ${dqc_tool_side / 2}" rpy="0 0 0"/>
         <geometry><cylinder radius="0.036" length="${dqc_tool_side}"/></geometry>
-        <material name="dqc_tool_side"><color rgba="0.15 0.35 0.75 1"/></material>
+        <material name="dqc_tool_side"><color rgba="0.35 0.45 0.6 1"/></material>
       </visual>
       <visual>
@@ -65,5 +65,7 @@
                 scale="0.001 0.001 0.001"/>
         </geometry>
-        <material name="soft_gripper_blue"><color rgba="0.3 0.45 0.95 1"/></material>
+        <!-- Blue-grey, not the real saturated blue: in Gazebo the colour
+             detector would otherwise take it for "the blue block". -->
+        <material name="soft_gripper_blue"><color rgba="0.4 0.6 0.85 1"/></material>
       </visual>
       <collision>
