Commit message: Gazebo + RViz: mount the RG2 on the Dual Quick Changer, add the changer and soft gripper
Shared ur7e_bringup/urdf/dual_quick_changer.xacro (CAD meshes for display,
padded boxes for collision) used by the Gazebo robot and by the MoveIt model
it plans with (which RViz draws). The RG2 sits on the 60 deg face; MoveIt's
group still ends at gripper_tcp, so every top-down goal now points the RG2,
not the flange, down. Allowed-collision pairs for the bolted-together parts.

Verified in Gazebo: language pick ok, pick_object lifted to z 0.140 m,
gripper_tcp RPY (180, 0, 0), tool0 pitched 60 deg. A test keeps the xacro
numbers equal to scripts/lab_tooling.py. Docs: Gazebo section in START_HERE,
stale latch claim in the Gazebo README corrected.

Co-Authored-By: Claude Opus 5.5 <noreply@anthropic.com>

File: src/ur7e_gazebo/urdf/ur7e_gz.urdf.xacro (robot description, xacro)
@@ -46,4 +46,5 @@
   <xacro:property name="prefix" value="$(arg tf_prefix)"/>
   <xacro:include filename="$(find onrobot_description)/urdf/rg2_macro.xacro"/>
+  <xacro:include filename="$(find ur7e_bringup)/urdf/dual_quick_changer.xacro"/>
   <link name="world"/>
   <xacro:ur_robot
@@ -106,9 +107,13 @@
   </joint>
   <xacro:finger_joints prefix="${prefix}" fingerprefix="left" reflect="1.0"/>
+  <!-- 2026-10-08: the RG2 sits on a face of the OnRobot Dual Quick Changer,
+       60 deg off the flange axis, not on tool0's axis; the changer and the
+       soft gripper on its other face come with it (dual_quick_changer.xacro). -->
   <joint name="$(arg tf_prefix)onrobot_base_link_joint" type="fixed">
     <parent link="$(arg tf_prefix)tool0"/>
     <child link="$(arg tf_prefix)onrobot_base_link"/>
-    <origin xyz="0 0 0" rpy="0 0 ${-pi/2}"/>
+    <xacro:rg2_on_dual_quick_changer_origin/>
   </joint>
+  <xacro:dual_quick_changer prefix="$(arg tf_prefix)"/>
   <!--
   Root cause #3 of the DetachableJoint saga (see this file's header + the

File: src/ur7e_pick_place_bringup/srdf/ur7e_pick_place.srdf.xacro (robot description, xacro)
@@ -30,3 +30,21 @@
     <joint name="$(arg prefix)wrist_3_joint" value="0"/>
   </group_state>
+  <!-- 2026-10-08: the Dual Quick Changer and the soft gripper
+       (ur7e_bringup/urdf/dual_quick_changer.xacro) are bolted to the flange
+       and to the RG2's base: touching each other is the mounting, not a
+       collision. Everything else (forearm, table, the RG2's fingers) is checked. -->
+  <disable_collisions link1="$(arg prefix)lab_changer" link2="$(arg prefix)tool0" reason="Adjacent"/>
+  <disable_collisions link1="$(arg prefix)lab_changer" link2="$(arg prefix)flange" reason="Adjacent"/>
+  <disable_collisions link1="$(arg prefix)lab_changer" link2="$(arg prefix)wrist_3_link" reason="Adjacent"/>
+  <disable_collisions link1="$(arg prefix)lab_changer" link2="$(arg prefix)wrist_2_link" reason="Adjacent"/>
+  <disable_collisions link1="$(arg prefix)lab_changer" link2="$(arg prefix)onrobot_base_link" reason="Adjacent"/>
+  <disable_collisions link1="$(arg prefix)lab_changer" link2="$(arg prefix)cable_connector_0" reason="Adjacent"/>
+  <disable_collisions link1="$(arg prefix)lab_changer" link2="$(arg prefix)cable_connector_1" reason="Adjacent"/>
+  <disable_collisions link1="$(arg prefix)lab_changer" link2="$(arg prefix)lab_soft_gripper" reason="Adjacent"/>
+  <disable_collisions link1="$(arg prefix)lab_soft_gripper" link2="$(arg prefix)tool0" reason="Adjacent"/>
+  <disable_collisions link1="$(arg prefix)lab_soft_gripper" link2="$(arg prefix)flange" reason="Adjacent"/>
+  <disable_collisions link1="$(arg prefix)lab_soft_gripper" link2="$(arg prefix)wrist_3_link" reason="Adjacent"/>
+  <disable_collisions link1="$(arg prefix)lab_soft_gripper" link2="$(arg prefix)onrobot_base_link" reason="Adjacent"/>
+  <disable_collisions link1="$(arg prefix)lab_soft_gripper" link2="$(arg prefix)cable_connector_0" reason="Adjacent"/>
+  <disable_collisions link1="$(arg prefix)lab_soft_gripper" link2="$(arg prefix)cable_connector_1" reason="Adjacent"/>
 </robot>

File: src/ur7e_pick_place_bringup/urdf/ur7e_pick_place.urdf.xacro (robot description, xacro)
@@ -24,22 +24,53 @@
   <xacro:arg name="input_recipe_filename" default="$(find ur_robot_driver)/resources/rtde_input_recipe.txt"/>
   <xacro:arg name="output_recipe_filename" default="$(find ur_robot_driver)/resources/rtde_output_recipe.txt"/>
-  <xacro:include filename="$(find ur_onrobot_description)/urdf/ur_onrobot_macro.xacro"/>
+  <!-- 2026-10-08: the vendored ur_onrobot macro bolts the RG2 to tool0 on
+       the flange axis. The real arm has an OnRobot Dual Quick Changer in
+       between (RG2 60 deg off axis, soft gripper on the other face), so its
+       body is expanded here with that mount; the vendored file is untouched.
+       Gazebo uses the same dual_quick_changer.xacro. -->
+  <xacro:include filename="$(find ur_description)/urdf/ur_macro.xacro"/>
+  <xacro:include filename="$(find onrobot_description)/urdf/onrobot_macro.xacro"/>
+  <xacro:include filename="$(find ur7e_bringup)/urdf/dual_quick_changer.xacro"/>
   <link name="world"/>
-  <xacro:ur_onrobot
+  <xacro:ur_robot
+      robot_ip="$(arg robot_ip)"
+      name="$(arg ur_type)"
       parent="world"
-      robot_ip="$(arg robot_ip)"
-      ur_type="$(arg ur_type)"
-      onrobot_type="$(arg onrobot_type)"
       tf_prefix="$(arg tf_prefix)"
       use_fake_hardware="$(arg use_fake_hardware)"
+      joint_limits_parameters_file="$(arg joint_limits_parameters_file)"
       kinematics_parameters_file="$(arg kinematics_parameters_file)"
-      joint_limits_parameters_file="$(arg joint_limits_parameters_file)"
       physical_parameters_file="$(arg physical_parameters_file)"
       visual_parameters_file="$(arg visual_parameters_file)"
       script_filename="$(arg script_filename)"
+      output_recipe_filename="$(arg output_recipe_filename)"
       input_recipe_filename="$(arg input_recipe_filename)"
-      output_recipe_filename="$(arg output_recipe_filename)"
       >
       <origin xyz="0 0 0" rpy="0 0 0" />
-  </xacro:ur_onrobot>
+  </xacro:ur_robot>
+  <xacro:onrobot onrobot_type="$(arg onrobot_type)" prefix="$(arg tf_prefix)"
+                 use_fake_hardware="$(arg use_fake_hardware)"/>
+  <joint name="$(arg tf_prefix)onrobot_base_link_joint" type="fixed">
+    <parent link="$(arg tf_prefix)tool0"/>
+    <child link="$(arg tf_prefix)onrobot_base_link"/>
+    <xacro:rg2_on_dual_quick_changer_origin/>
+  </joint>
+  <xacro:dual_quick_changer prefix="$(arg tf_prefix)"/>
+  <!-- Cable connectors on the RG2, as in the vendored macro (its SRDF names them). -->
+  <link name="$(arg tf_prefix)cable_connector_0">
+    <collision><geometry><sphere radius="0.03"/></geometry></collision>
+  </link>
+  <joint name="$(arg tf_prefix)cable_connector_0_joint" type="fixed">
+    <parent link="$(arg tf_prefix)onrobot_base_link"/>
+    <child link="$(arg tf_prefix)cable_connector_0"/>
+    <origin xyz="0 -0.035 0.01" rpy="0 0 0"/>
+  </joint>
+  <link name="$(arg tf_prefix)cable_connector_1">
+    <collision><geometry><sphere radius="0.03"/></geometry></collision>
+  </link>
+  <joint name="$(arg tf_prefix)cable_connector_1_joint" type="fixed">
+    <parent link="$(arg tf_prefix)onrobot_base_link"/>
+    <child link="$(arg tf_prefix)cable_connector_1"/>
+    <origin xyz="0.03 0.0 -0.03" rpy="0 0 0"/>
+  </joint>
 </robot>

Commit message: Chess arm: single RG2 on a new UR, board calibration, camera vision, live dashboard
The chess match runs on a different UR (calibration hash calib_3365807260068553006,
192.168.1.10) with one RG2 bolted straight to the flange; the project-1 arm and
its Dual Quick Changer stay supported behind switches.

Arm and gripper
- tool_mount single|dual (xacro arg, default single) and mount: in
  lab_tooling.yaml; Gazebo, MoveIt URDF/SRDF and the lab planner follow it.
- ROBOT_IP / LAPTOP_IP / RG2_SERIAL / UR_LINK env vars (defaults unchanged),
  forwarded by the devcontainer; RG2 found by serial, not tool index.
- New factory kinematics for this arm (ur7e_calibration.yaml).
- Devcontainer base image default moved into the Dockerfile:
  ${localEnv:VAR:default} cut "osrf/ros:humble-desktop-full" at its first ':'.

Board calibration (lab_chess.py)
- fit --square (true square nearest the touches, keeps the tilt), board as a
  plane (0.8 deg tilt measured), mirrored-corner check, board thickness from a
  ruler instead of the project-1 table, teach-home beside the board.
- overlay: camera pose from the board grid (partial grids, CLAHE, retries,
  colour + last-pose disambiguation); watch: live view with target verdict.

Camera in the loop (chess_vision.py, OpenCV stereo, no ZED SDK)
- Lens tilt re-fitted per session; disparity offset measured on the board
  every scan (was 39.6 px); heights +-1.4 mm; pieces as 3-D clusters per
  square, robot cut out, nothing above 11 cm.
- scan, track [--apply] (board slide/turn with the camera fixed),
  move/play --vision (pick at the seen centre, grip at 3/4 measured height,
  student's move read from the board, board checked after arm moves).
- Empty-close threshold 12.3 mm (RG2 reads 9.3 closed on nothing).
- Browser dashboard served by watch: status line, game record vs camera
  boards, arm stage stepper, camera check, moves.

Lab-tested 2026-10-10/11: calibration, vision picks, a game started with the
camera reading the student's moves.

Co-Authored-By: Claude Opus 5.5 <noreply@anthropic.com>

File: src/ur7e_gazebo/urdf/ur7e_gz.urdf.xacro (robot description, xacro)
@@ -33,4 +33,7 @@
   <xacro:arg name="ur_type" default="ur7e"/>
   <xacro:arg name="tf_prefix" default=""/>
+  <!-- single: RG2 straight on the flange (chess arm); dual: Dual Quick Changer
+       (project-1 arm). Must match scripts/lab_tooling.yaml's mount. -->
+  <xacro:arg name="tool_mount" default="single"/>
   <xacro:arg name="kinematics_parameters_file"
              default="$(find ur7e_bringup)/config/ur7e_calibration.yaml"/>
@@ -113,7 +116,8 @@
     <parent link="$(arg tf_prefix)tool0"/>
     <child link="$(arg tf_prefix)onrobot_base_link"/>
-    <xacro:rg2_on_dual_quick_changer_origin/>
+    <xacro:if value="${'$(arg tool_mount)' == 'dual'}"><xacro:rg2_on_dual_quick_changer_origin/></xacro:if>
+    <xacro:unless value="${'$(arg tool_mount)' == 'dual'}"><origin xyz="0 0 0" rpy="0 0 ${-pi/2}"/></xacro:unless>
   </joint>
-  <xacro:dual_quick_changer prefix="$(arg tf_prefix)"/>
+  <xacro:if value="${'$(arg tool_mount)' == 'dual'}"><xacro:dual_quick_changer prefix="$(arg tf_prefix)"/></xacro:if>
   <!--
   Root cause #3 of the DetachableJoint saga (see this file's header + the

File: src/ur7e_pick_place_bringup/srdf/ur7e_pick_place.srdf.xacro (robot description, xacro)
@@ -13,4 +13,7 @@
   <xacro:arg name="name" default="ur_onrobot"/>
   <xacro:arg name="prefix" default=""/>
+  <!-- single: RG2 straight on the flange (chess arm); dual: Dual Quick Changer
+       (project-1 arm). Must match scripts/lab_tooling.yaml's mount. -->
+  <xacro:arg name="tool_mount" default="single"/>
   <xacro:include filename="$(find ur_onrobot_moveit_config)/srdf/ur_onrobot_macro.srdf.xacro"/>
   <xacro:ur_onrobot_srdf name="$(arg name)" prefix="$(arg prefix)"/>
@@ -34,17 +37,19 @@
        and to the RG2's base: touching each other is the mounting, not a
        collision. Everything else (forearm, table, the RG2's fingers) is checked. -->
-  <disable_collisions link1="$(arg prefix)lab_changer" link2="$(arg prefix)tool0" reason="Adjacent"/>
-  <disable_collisions link1="$(arg prefix)lab_changer" link2="$(arg prefix)flange" reason="Adjacent"/>
-  <disable_collisions link1="$(arg prefix)lab_changer" link2="$(arg prefix)wrist_3_link" reason="Adjacent"/>
-  <disable_collisions link1="$(arg prefix)lab_changer" link2="$(arg prefix)wrist_2_link" reason="Adjacent"/>
-  <disable_collisions link1="$(arg prefix)lab_changer" link2="$(arg prefix)onrobot_base_link" reason="Adjacent"/>
-  <disable_collisions link1="$(arg prefix)lab_changer" link2="$(arg prefix)cable_connector_0" reason="Adjacent"/>
-  <disable_collisions link1="$(arg prefix)lab_changer" link2="$(arg prefix)cable_connector_1" reason="Adjacent"/>
-  <disable_collisions link1="$(arg prefix)lab_changer" link2="$(arg prefix)lab_soft_gripper" reason="Adjacent"/>
-  <disable_collisions link1="$(arg prefix)lab_soft_gripper" link2="$(arg prefix)tool0" reason="Adjacent"/>
-  <disable_collisions link1="$(arg prefix)lab_soft_gripper" link2="$(arg prefix)flange" reason="Adjacent"/>
-  <disable_collisions link1="$(arg prefix)lab_soft_gripper" link2="$(arg prefix)wrist_3_link" reason="Adjacent"/>
-  <disable_collisions link1="$(arg prefix)lab_soft_gripper" link2="$(arg prefix)onrobot_base_link" reason="Adjacent"/>
-  <disable_collisions link1="$(arg prefix)lab_soft_gripper" link2="$(arg prefix)cable_connector_0" reason="Adjacent"/>
-  <disable_collisions link1="$(arg prefix)lab_soft_gripper" link2="$(arg prefix)cable_connector_1" reason="Adjacent"/>
+  <xacro:if value="${'$(arg tool_mount)' == 'dual'}">
+    <disable_collisions link1="$(arg prefix)lab_changer" link2="$(arg prefix)tool0" reason="Adjacent"/>
+    <disable_collisions link1="$(arg prefix)lab_changer" link2="$(arg prefix)flange" reason="Adjacent"/>
+    <disable_collisions link1="$(arg prefix)lab_changer" link2="$(arg prefix)wrist_3_link" reason="Adjacent"/>
+    <disable_collisions link1="$(arg prefix)lab_changer" link2="$(arg prefix)wrist_2_link" reason="Adjacent"/>
+    <disable_collisions link1="$(arg prefix)lab_changer" link2="$(arg prefix)onrobot_base_link" reason="Adjacent"/>
+    <disable_collisions link1="$(arg prefix)lab_changer" link2="$(arg prefix)cable_connector_0" reason="Adjacent"/>
+    <disable_collisions link1="$(arg prefix)lab_changer" link2="$(arg prefix)cable_connector_1" reason="Adjacent"/>
+    <disable_collisions link1="$(arg prefix)lab_changer" link2="$(arg prefix)lab_soft_gripper" reason="Adjacent"/>
+    <disable_collisions link1="$(arg prefix)lab_soft_gripper" link2="$(arg prefix)tool0" reason="Adjacent"/>
+    <disable_collisions link1="$(arg prefix)lab_soft_gripper" link2="$(arg prefix)flange" reason="Adjacent"/>
+    <disable_collisions link1="$(arg prefix)lab_soft_gripper" link2="$(arg prefix)wrist_3_link" reason="Adjacent"/>
+    <disable_collisions link1="$(arg prefix)lab_soft_gripper" link2="$(arg prefix)onrobot_base_link" reason="Adjacent"/>
+    <disable_collisions link1="$(arg prefix)lab_soft_gripper" link2="$(arg prefix)cable_connector_0" reason="Adjacent"/>
+    <disable_collisions link1="$(arg prefix)lab_soft_gripper" link2="$(arg prefix)cable_connector_1" reason="Adjacent"/>
+  </xacro:if>
 </robot>

File: src/ur7e_pick_place_bringup/urdf/ur7e_pick_place.urdf.xacro (robot description, xacro)
@@ -11,4 +11,7 @@
   <xacro:arg name="ur_type" default="ur7e"/>
   <xacro:arg name="onrobot_type" default="rg2"/>
+  <!-- single: RG2 straight on the flange (chess arm); dual: Dual Quick Changer
+       (project-1 arm). Must match scripts/lab_tooling.yaml's mount. -->
+  <xacro:arg name="tool_mount" default="single"/>
   <xacro:arg name="tf_prefix" default=""/>
   <xacro:arg name="use_fake_hardware" default="true"/>
@@ -54,7 +57,8 @@
     <parent link="$(arg tf_prefix)tool0"/>
     <child link="$(arg tf_prefix)onrobot_base_link"/>
-    <xacro:rg2_on_dual_quick_changer_origin/>
+    <xacro:if value="${'$(arg tool_mount)' == 'dual'}"><xacro:rg2_on_dual_quick_changer_origin/></xacro:if>
+    <xacro:unless value="${'$(arg tool_mount)' == 'dual'}"><origin xyz="0 0 0" rpy="0 0 ${-pi/2}"/></xacro:unless>
   </joint>
-  <xacro:dual_quick_changer prefix="$(arg tf_prefix)"/>
+  <xacro:if value="${'$(arg tool_mount)' == 'dual'}"><xacro:dual_quick_changer prefix="$(arg tf_prefix)"/></xacro:if>
   <!-- Cable connectors on the RG2, as in the vendored macro (its SRDF names them). -->
   <link name="$(arg tf_prefix)cable_connector_0">
